Commit message: manual xform calc

File: src/basic_mobile_robot/models/edward_the_robot.urdf (robot description, URDF)
Before this commit: robot edward, 31 links, 30 joints
Links:
- removed link camera_depth_frame
- removed link camera_depth_optical_frame
- removed link camera_link
- removed link camera_rgb_frame
- removed link camera_rgb_optical_frame
Joints:
- removed joint camera_depth_joint
- removed joint camera_depth_optical_joint
- removed joint camera_joint
- removed joint camera_rgb_optical_joint

Commit message: Added Parameters

File: src/basic_mobile_robot/models/edward_the_robot.urdf (robot description, URDF)
Before this commit: robot edward, 26 links, 26 joints
Links:
- added link camera_depth_frame, mass 0.001; visual sphere radius=0.015
- added link camera_depth_optical_frame, mass 0.001
- added link camera_link
- added link camera_rgb_frame, mass 0.001; visual sphere radius=0.02
- added link camera_rgb_optical_frame, mass 0.001
Joints:
- added joint camera_depth_joint: type fixed, parent camera_rgb_frame, child camera_depth_frame, origin xyz=0 0.0 0 rpy=0 0 0
- added joint camera_depth_optical_joint: type fixed, parent camera_depth_frame, child camera_depth_optical_frame, origin xyz=0 0.0 0 rpy=-1.57079632679 0 -1.57079632679
- added joint camera_joint: type fixed, parent camera_link, child camera_rgb_frame, origin xyz=0.0 -0.0 -0.0 rpy=-1.570795 0 -1.570795
- added joint camera_rgb_optical_joint: type fixed, parent camera_rgb_frame, child camera_rgb_optical_frame, origin xyz=0 0 0 rpy=-1.57079632679 0 -1.57079632679
